File: KICAD files/splitkbright/splitkb.kicad_pcb (KiCad board)
At the start: 2 copper layers, 131.3 x 114.6 mm, 83 parts, among them SW31 SW_Push, SW32 SW_Push, SW37 SW_Push, SW38 SW_Push, SW39 SW_Push, SW40 SW_Push, SW41 SW_Push, SW42 SW_Push, SW43 SW_Push, SW44 SW_Push, SW45 SW_Push, SW46 SW_Push, SW47 SW_Push, SW48 SW_Push, SW49 SW_Push, SW50 SW_Push, SW51 SW_Push, SW52 SW_Push, SW53 SW_Push, SW54 SW_Push, SW55 SW_Push, SW56 SW_Push, SW57 SW_Push, SW58 SW_Push, SW59 SW_Push, SW60 SW_Push, SW61 SW_Push, SW62 SW_Push, SW63 SW_Push, SW64 SW_Push, SW65 SW_Push, SW66 SW_Push, SW67 SW_Push, SW68 SW_Push, SW69 SW_Push, SW70 SW_Push, SW71 SW_Push, SW72 SW_Push, SW73 SW_Push, SW74 SW_Push, U1 nice_nano

Commit message: Ran new traces and moved controller
Parts:
- moved U1 6.10 mm to (247.9, 136.0)
Routing:
- net row4: track 138.1 -> 132.0 mm
- net col6: track 96.8 -> 90.7 mm
- net col4: track 126.7 -> 132.8 mm
- net col3: track 150.0 -> 156.1 mm
- net col2: track 167.3 -> 173.4 mm
- net col0: track 212.8 -> 218.9 mm
- net col1: track 194.2 -> 200.3 mm
- net row1: track 211.8 -> 206.0 mm
- net row5: track 85.6 -> 91.4 mm
- net GND: track 74.9 -> 69.7 mm
- net row0: track 229.2 -> 224.2 mm
- net bat: track 77.4 -> 73.2 mm
- net row2: track 182.9 -> 179.4 mm
- net row3: track 161.9 -> 164.6 mm
- net col5: track 101.9 -> 104.5 mm
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