File: KICAD files/splitkbright/untitled.kicad_sch (KiCad schematic)
At the start: 75 parts, among them SW1 SW_Push, SW10 SW_Push, SW11 SW_Push, SW12 SW_Push, SW13 SW_Push, SW14 SW_Push, SW15 SW_Push, SW16 SW_Push, SW17 SW_Push, SW18 SW_Push, SW19 SW_Push, SW2 SW_Push, SW20 SW_Push, SW21 SW_Push, SW22 SW_Push, SW23 SW_Push, SW24 SW_Push, SW25 SW_Push, SW26 SW_Push, SW27 SW_Push, SW28 SW_Push, SW29 SW_Push, SW3 SW_Push, SW30 SW_Push, SW31 SW_Push, SW32 SW_Push, SW33 SW_Push, SW34 SW_Push, SW4 SW_Push, SW5 SW_Push, SW6 SW_Push, SW7 SW_Push, SW8 SW_Push, SW9 SW_Push, U1 NRF52840

Commit message: Edited PCB.
- Changed the footprint used for the dev board.
- Ran traces again for the dev board.
- Made a custom symbol and footprint for the devboard.
Parts:
- removed U1: NRF52840, nice-nano-kicad-master:NRF52840, symbol NRF52840_library:NRF52840
- added U2: NRF52840, nice-nano-kicad-master:NRF52840, symbol NRF52840_library:NRF52840
- renumbered D2 to D1, D18 to D10, D24 to D11, D3 to D12, D8 to D13, D13 to D14, D19 to D15, D25 to D16, D4 to D17, D9 to D18, D14 to D19, D1 to D2, D26 to D21, D5 to D22, D10 to D23, D15 to D24, D21 to D25, D27 to D26, D32 to D27, D33 to D28, D30 to D29, D6 to D3, D31 to D30, D16 to D33, D22 to D34, D28 to D35, D34 to D36, D11 to D4, D17 to D5, D23 to D6, D29 to D7, D7 to D8, D12 to D9, H1 to H5, H2 to H6, H3 to H7, H4 to H8, SW18 to SW10, SW24 to SW11, SW30 to SW12, SW3 to SW13, SW8 to SW14, SW13 to SW15, SW19 to SW16, SW25 to SW17, SW31 to SW18, SW4 to SW19, SW6 to SW2, SW9 to SW20, SW14 to SW21, SW20 to SW22, SW26 to SW23, SW32 to SW24, SW5 to SW25, SW10 to SW26, SW15 to SW27, SW21 to SW28, SW27 to SW29, SW11 to SW3, SW33 to SW30, SW16 to SW33, SW22 to SW34, SW28 to SW35, SW34 to SW36, SW17 to SW4, SW23 to SW5, SW29 to SW6, SW2 to SW7, SW7 to SW8, SW12 to SW9, TP1 to TP3, TP2 to TP4
Connections:
- net GND: now also U2.24 (GND)
- net bat: now also U2.26 (BAT+)
- net col0: now also U2.2 (D1/P0.06)
- net col1: now also U2.3 (D0/P0.08)
- net col2: now also U2.6 (D2/P0.17)
- net col3: now also U2.7 (D3/P0.20)
- net col4: now also U2.8 (D4/P0.22)
- net col5: now also U2.9 (D5/P0.24)
- net row0: now also U2.10 (D6/P1.00)
- net row1: now also U2.11 (D7/P0.11)
- net row2: now also U2.12 (D8/P1.04)
- net row3: now also U2.13 (D9/P1.06)
- net row4: now also U2.14 (D10/P0.09)
- net row5: now also U2.15 (D16/P0.10)
