File: KICAD files/splitkbright/splitkb.kicad_sch (KiCad schematic)
At the start: 4 parts

Commit message: Cleaned up the kicad project.
Other:
- sheet left: file untitled.kicad_sch -> left.kicad_sch
Changed lines of the file:
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@@
 			)
 		)
-		(property "Sheetfile" "untitled.kicad_sch"
+		(property "Sheetfile" "left.kicad_sch"
 			(at 171.45 105.9946 0)
 			(show_name no)
