File: KICAD files/splitkbleft/splitkbleft.kicad_pcb (KiCad board)
At the start: 2 copper layers, 114.8 x 116.8 mm, 71 parts, among them SW1 SW_Push, SW10 SW_Push, SW11 SW_Push, SW12 SW_Push, SW13 SW_Push, SW14 SW_Push, SW15 SW_Push, SW16 SW_Push, SW17 SW_Push, SW18 SW_Push, SW19 SW_Push, SW2 SW_Push, SW20 SW_Push, SW21 SW_Push, SW22 SW_Push, SW23 SW_Push, SW24 SW_Push, SW25 SW_Push, SW26 SW_Push, SW27 SW_Push, SW28 SW_Push, SW29 SW_Push, SW3 SW_Push, SW30 SW_Push, SW33 SW_Push, SW34 SW_Push, SW35 SW_Push, SW36 SW_Push, SW4 SW_Push, SW5 SW_Push, SW6 SW_Push, SW7 SW_Push, SW8 SW_Push, SW9 SW_Push, U2 nice_nano

Commit message: Edited PCBs
- Added mounting holes to both pcbs and schematics
- Changed the shape and size of both PCBs
Parts:
- added REF**: MountingHole_2.2mm_M2, MountingHole:MountingHole_2.2mm_M2, F.Cu at (165.1, 162.1)
- added REF**: MountingHole_2.2mm_M2, MountingHole:MountingHole_2.2mm_M2, F.Cu at (75.7, 57.9)
- added REF**: MountingHole_2.2mm_M2, MountingHole:MountingHole_2.2mm_M2, F.Cu at (166.6, 55.9)
- added REF**: MountingHole_2.2mm_M2, MountingHole:MountingHole_2.2mm_M2, F.Cu at (57.4, 167.6)
- moved U2 2.70 mm to (72.9, 156.4)
Routing:
- net row2: track 182.7 -> 172.8 mm, vias 2 -> 1
- net row1: track 199.8 -> 190.7 mm, vias 2 -> 1
- net bat: track 193.6 -> 196.5 mm
- net GND: track 194.2 -> 197.0 mm
- net col2: track 114.8 -> 117.5 mm
- net row5: track 142.3 -> 145.0 mm
- net row0: track 216.0 -> 218.4 mm
- net col1: track 97.5 -> 99.5 mm
- net col3: track 149.8 -> 151.7 mm
- net col4: track 161.6 -> 162.7 mm
- net col0: track 87.3 -> 88.5 mm
- net row3: track 133.7 -> 133.0 mm
- net row4: track 194.8 -> 195.5 mm
- net col5: track 176.6 -> 177.2 mm
Other:
- board size 114.8 x 116.8 mm -> 114.8 x 120.4 mm
